Commit message: mimic joint action; ground friction; foot box collision

File: source/g1_hoi_learning/g1_hoi_learning/assets/unitree_g1/g1_29dof_rev_1_0_with_inspire_hand_DFQ.urdf (robot description, URDF)
Before this commit: robot g1_29dof_rev_1_0_with_inspire_hand_DFQ, 73 links, 72 joints
Links:
- link left_ankle_roll_link: geometry collision box size=0.186 0.072 0.020; visual mesh filename=meshes/left_ankle_roll_link.STL
- link right_ankle_roll_link: geometry collision box size=0.186 0.072 0.020; visual mesh filename=meshes/right_ankle_roll_link.STL
